File: hw-design/Power.sch (KiCad schematic (older format))
At the start: 15 parts, among them U2 AP1117E50G, U3 AP1117E33G

Commit message: moving I/O stuff to new sheet
Parts:
- added CN1, CN2: CONN_PANNEL_2X2, MOD_Footprints_Lib:CONN_PANNEL, symbol CONN_PANNEL_2X2
Connections:
- wire segments 38 -> 50
Changed lines of the file:
@@
 LIBS:MOD_PEX_Prototype1
 LIBS:Duo_Audio_HMI_RC1A
-LIBS:MOD_PEX_Prototype1-cache
+LIBS:expression-pedal-cache
 EELAYER 25 0
 EELAYER END
 $Descr A4 11693 8268
 encoding utf-8
-Sheet 2 4
+Sheet 2 5
 Title ""
 Date ""
@@
 $EndComp
 $Comp
-L DGND #PWR013
+L DGND #PWR01
 U 1 1 548B65EB
 P 6650 4100
-F 0 "#PWR013" H 6650 4100 40  0001 C CNN
+F 0 "#PWR01" H 6650 4100 40  0001 C CNN
 F 1 "DGND" H 6650 4030 40  0000 C CNN
 F 2 "" H 6650 4100 60  0000 C CNN
@@
 $EndComp
 $Comp
-L DGND #PWR014
+L DGND #PWR02
 U 1 1 548B65F1
 P 5350 4100
-F 0 "#PWR014" H 5350 4100 40  0001 C CNN
+F 0 "#PWR02" H 5350 4100 40  0001 C CNN
 F 1 "DGND" H 5350 4030 40  0000 C CNN
 F 2 "" H 5350 4100 60  0000 C CNN
@@
 $EndComp
 $Comp
-L DGND #PWR015
+L DGND #PWR03
 U 1 1 548B65FE
 P 6050 3900
-F 0 "#PWR015" H 6050 3900 40  0001 C CNN
+F 0 "#PWR03" H 6050 3900 40  0001 C CNN
 F 1 "DGND" H 6050 3830 40  0000 C CNN
 F 2 "" H 6050 3900 60  0000 C CNN
@@
 $EndComp
 $Comp
-L +3.3V #PWR016
+L +3.3V #PWR04
 U 1 1 548B6604
 P 7600 3350
-F 0 "#PWR016" H 7600 3310 30  0001 C CNN
+F 0 "#PWR04" H 7600 3310 30  0001 C CNN
 F 1 "+3.3V" H 7600 3460 30  0000 C CNN
 F 2 "" H 7600 3350 60  0000 C CNN
@@
 $EndComp
 $Comp
-L DGND #PWR017
+L DGND #PWR05
 U 1 1 548B6611
 P 6900 4100
-F 0 "#PWR017" H 6900 4100 40  0001 C CNN
+F 0 "#PWR05" H 6900 4100 40  0001 C CNN
 F 1 "DGND" H 6900 4030 40  0000 C CNN
 F 2 "" H 6900 4100 60  0000 C CNN
@@
 $EndComp
 $Comp
-L PWR_FLAG #FLG018
+L PWR_FLAG #FLG06
 U 1 1 548B661E
 P 7800 3400
-F 0 "#FLG018" H 7800 3495 30  0001 C CNN
+F 0 "#FLG06" H 7800 3495 30  0001 C CNN
 F 1 "PWR_FLAG" H 7800 3580 30  0000 C CNN
 F 2 "" H 7800 3400 60  0000 C CNN
@@
 $EndComp
 $Comp
-L DGND #PWR019
+L DGND #PWR07
 U 1 1 548B662B
 P 5600 4100
-F 0 "#PWR019" H 5600 4100 40  0001 C CNN
+F 0 "#PWR07" H 5600 4100 40  0001 C CNN
 F 1 "DGND" H 5600 4030 40  0000 C CNN
 F 2 "" H 5600 4100 60  0000 C CNN
@@
 $EndComp
 $Comp
-L DGND #PWR020
+L DGND #PWR08
 U 1 1 548B6638
 P 4050 4100
-F 0 "#PWR020" H 4050 4100 40  0001 C CNN
+F 0 "#PWR08" H 4050 4100 40  0001 C CNN
 F 1 "DGND" H 4050 4030 40  0000 C CNN
 F 2 "" H 4050 4100 60  0000 C CNN
@@
 $EndComp
 $Comp
-L +9V #PWR021
+L +9V #PWR09
 U 1 1 548B6645
 P 4050 3350
-F 0 "#PWR021" H 4050 3320 20  0001 C CNN
+F 0 "#PWR09" H 4050 3320 20  0001 C CNN
 F 1 "+9V" H 4050 3460 30  0000 C CNN
 F 2 "" H 4050 3350 60  0000 C CNN
@@
 $EndComp
 $Comp
-L VCC #PWR022
+L VCC #PWR010
 U 1 1 548B664B
 P 2750 3400
-F 0 "#PWR022" H 2750 3500 30  0001 C CNN
+F 0 "#PWR010" H 2750 3500 30  0001 C CNN
 F 1 "VCC" H 2750 3500 30  0000 C CNN
 F 2 "" H 2750 3400 60  0000 C CNN
@@
 $EndComp
 $Comp
-L DGND #PWR023
+L DGND #PWR011
 U 1 1 548B6666
 P 4300 4100
-F 0 "#PWR023" H 4300 4100 40  0001 C CNN
+F 0 "#PWR011" H 4300 4100 40  0001 C CNN
 F 1 "DGND" H 4300 4030 40  0000 C CNN
 F 2 "" H 4300 4100 60  0000 C CNN
@@
 $EndComp
 $Comp
-L PWR_FLAG #FLG024
+L PWR_FLAG #FLG012
 U 1 1 548B666C
 P 4300 3400
-F 0 "#FLG024" H 4300 3495 30  0001 C CNN
+F 0 "#FLG012" H 4300 3495 30  0001 C CNN
 F 1 "PWR_FLAG" H 4300 3580 30  0000 C CNN
 F 2 "" H 4300 3400 60  0000 C CNN
@@
 $EndComp
 $Comp
-L +5V #PWR025
+L +5V #PWR013
 U 1 1 548B6672
 P 5350 2850
-F 0 "#PWR025" H 5350 2940 20  0001 C CNN
+F 0 "#PWR013" H 5350 2940 20  0001 C CNN
 F 1 "+5V" H 5350 2940 30  0000 C CNN
 F 2 "" H 5350 2850 60  0000 C CNN
@@
 $EndComp
 $Comp
-L DGND #PWR026
+L DGND #PWR014
 U 1 1 548B6678
 P 4750 3900
-F 0 "#PWR026" H 4750 3900 40  0001 C CNN
+F 0 "#PWR014" H 4750 3900 40  0001 C CNN
 F 1 "DGND" H 4750 3830 40  0000 C CNN
 F 2 "" H 4750 3900 60  0000 C CNN
@@
 Connection ~ 6550 3500
 $Comp
-L PWR_FLAG #FLG027
+L PWR_FLAG #FLG015
 U 1 1 548B66C1
 P 5500 2850
-F 0 "#FLG027" H 5500 2945 30  0001 C CNN
+F 0 "#FLG015" H 5500 2945 30  0001 C CNN
 F 1 "PWR_FLAG" H 5500 3030 30  0000 C CNN
 F 2 "" H 5500 2850 60  0000 C CNN
@@
 Connection ~ 3250 3500
 $Comp
-L PWR_FLAG #FLG028
+L PWR_FLAG #FLG016
 U 1 1 54B500E8
 P 3650 3950
-F 0 "#FLG028" H 3650 4045 30  0001 C CNN
+F 0 "#FLG016" H 3650 4045 30  0001 C CNN
 F 1 "PWR_FLAG" H 3650 4130 30  0000 C CNN
 F 2 "" H 3650 3950 60  0000 C CNN
@@
 $EndComp
 $Comp
-L DGND #PWR029
+L DGND #PWR017
 U 1 1 54B50120
 P 3650 4100
-F 0 "#PWR029" H 3650 4100 40  0001 C CNN
+F 0 "#PWR017" H 3650 4100 40  0001 C CNN
 F 1 "DGND" H 3650 4030 40  0000 C CNN
 F 2 "" H 3650 4100 60  0000 C CNN
@@
 	3650 3950 3650 4100
 $Comp
-L PWR_FLAG #FLG030
+L PWR_FLAG #FLG018
 U 1 1 54B50E4C
 P 2450 3450
-F 0 "#FLG030" H 2450 3545 30  0001 C CNN
+F 0 "#FLG018" H 2450 3545 30  0001 C CNN
 F 1 "PWR_FLAG" H 2450 3630 30  0000 C CNN
 F 2 "" H 2450 3450 60  0000 C CNN
@@
 	2450 3450 2450 3500
 Connection ~ 2750 3500
+$Comp
+L CONN_PANNEL_2X2 CN1
+U 1 1 54CBF1DD
+P 2400 5800
+F 0 "CN1" H 2400 5950 50  0000 C CNN
+F 1 "CONN_PANNEL_2X2" H 2410 5670 40  0000 C CNN
+F 2 "MOD_Footprints_Lib:CONN_PANNEL" H 2400 5800 60  0001 C CNN
+F 3 "" H 2400 5800 60  0000 C CNN
+	1    2400 5800
+	1    0    0    -1
+$EndComp
+$Comp
+L CONN_PANNEL_2X2 CN2
+U 1 1 54CBF1E4
+P 3650 5800
+F 0 "CN2" H 3650 5950 50  0000 C CNN
+F 1 "CONN_PANNEL_2X2" H 3660 5670 40  0000 C CNN
+F 2 "MOD_Footprints_Lib:CONN_PANNEL" H 3650 5800 60  0001 C CNN
+F 3 "" H 3650 5800 60  0000 C CNN
+	1    3650 5800
+	1    0    0    -1
+$EndComp
+$Comp
+L DGND #PWR019
+U 1 1 54CBF1EB
+P 1950 5950
+F 0 "#PWR019" H 1950 5950 40  0001 C CNN
+F 1 "DGND" H 1950 5880 40  0000 C CNN
+F 2 "" H 1950 5950 60  0000 C CNN
+F 3 "" H 1950 5950 60  0000 C CNN
+	1    1950 5950
+	1    0    0    -1
+$EndComp
+Wire Wire Line
+	2000 5850 1950 5850
+Wire Wire Line
+	1950 5750 1950 5950
+Wire Wire Line
+	1950 5750 2000 5750
+Connection ~ 1950 5850
+$Comp
+L DGND #PWR020
+U 1 1 54CBF1F5
+P 2850 5950
+F 0 "#PWR020" H 2850 5950 40  0001 C CNN
+F 1 "DGND" H 2850 5880 40  0000 C CNN
+F 2 "" H 2850 5950 60  0000 C CNN
+F 3 "" H 2850 5950 60  0000 C CNN
+	1    2850 5950
+	1    0    0    -1
+$EndComp
+Wire Wire Line
+	2800 5850 2850 5850
+Wire Wire Line
+	2850 5750 2850 5950
+Wire Wire Line
+	2800 5750 2850 5750
+Connection ~ 2850 5850
+$Comp
+L DGND #PWR021
+U 1 1 54CBF1FF
+P 3200 5950
+F 0 "#PWR021" H 3200 5950 40  0001 C CNN
+F 1 "DGND" H 3200 5880 40  0000 C CNN
+F 2 "" H 3200 5950 60  0000 C CNN
+F 3 "" H 3200 5950 60  0000 C CNN
+	1    3200 5950
+	1    0    0    -1
+$EndComp
+$Comp
+L DGND #PWR022
+U 1 1 54CBF205
+P 4100 5950
+F 0 "#PWR022" H 4100 5950 40  0001 C CNN
+F 1 "DGND" H 4100 5880 40  0000 C CNN
+F 2 "" H 4100 5950 60  0000 C CNN
+F 3 "" H 4100 5950 60  0000 C CNN
+	1    4100 5950
+	1    0    0    -1
+$EndComp
+Wire Wire Line
+	4100 5750 4100 5950
+Wire Wire Line
+	4100 5850 4050 5850
+Wire Wire Line
+	4050 5750 4100 5750
+Connection ~ 4100 5850
+Wire Wire Line
+	3250 5850 3200 5850
+Wire Wire Line
+	3200 5750 3200 5950
+Wire Wire Line
+	3200 5750 3250 5750
+Connection ~ 3200 5850
 $EndSCHEMATC
