File: hw-design/expression-pedal.sch (KiCad schematic (older format))
At the start: 14 parts, among them CN1 CONN_PANNEL_2X2, CN2 CONN_PANNEL_2X2, P1 HEADER_3X1, P4 HEADER_2X1, SW1 SWITCH_HH

Commit message: moving I/O stuff to new sheet
Parts:
- removed C15, C9: 100nF_X7R, MOD_Footprints_Lib:SM0603, symbol C
- removed CN1, CN2: CONN_PANNEL_2X2, MOD_Footprints_Lib:CONN_PANNEL, symbol CONN_PANNEL_2X2
- removed P1: HEADER_3X1, MOD_Footprints_Lib:PIN_ARRAY_3X1, symbol CONN_3
- removed P4: HEADER_2X1, MOD_Footprints_Lib:PIN_ARRAY_2X1, symbol CONN_2
- removed R17, R18, R19: 100R, MOD_Footprints_Lib:SM0603, symbol R
- removed R23, R24, R25, R28: 10k, MOD_Footprints_Lib:SM0603, symbol R
- removed SW1: SWITCH_HH, MOD_Footprints_Lib:SWITCH_HH_SK-13D26-G-6_5-K-GY, symbol SWITCH_1-3
Connections:
- net labels removed: +3.3V, DGND, FOOT, POT, SW1, SW2, SW3
- wire segments 40 -> 0
Other:
- note removed: "FOOT"
- note removed: "POTENCIOMETER 10K"
- note removed: "SWITCH H-H"
