File: hw-design/cpu.sch (KiCad schematic (older format))
At the start: 17 parts, among them P2 HEADER_5X2, P3 HEADER_5X2, U1 LPC111X_LQFP48, X1 10MHz

Commit message: changing cpu schematic to use default kicad components library
Parts:
- removed R20: 10k, MOD_Footprints_Lib:SM0603, symbol R
- removed R22: 0R, MOD_Footprints_Lib:SM0603, symbol R
- removed U1: LPC111X_LQFP48, MOD_Footprints_Lib:LQFP48, symbol LPC111X_LQFP48
- added U1: LPC1113FBD48/302, LQFP48, symbol LPC1113FBD48/302
- C11, C12: value 18pF_NP0 -> 18pF X7R
- C13, C14: value 100nF_X7R -> 100nF X7R
Connections:
- net labels added: +3.3VP, GNDD
- net labels removed: +3.3V, +5V, DGND
- wire segments 68 -> 77
- no-connect marks 31 -> 32
Other:
- moved on the sheet: C10, C11, C12, C13, C14, R21, X1
