File: hw-design/io.sch (KiCad schematic (older format))
At the start: 12 parts, among them P1 HEADER_2X1, P4 HEADER_3X1, SW1 SWITCH_HH

Commit message: changing I/O schematic to use default kicad components library
Parts:
- removed P1: HEADER_2X1, MOD_Footprints_Lib:PIN_ARRAY_2X1, symbol CONN_2
- removed P4: HEADER_3X1, MOD_Footprints_Lib:PIN_ARRAY_3X1, symbol CONN_3
- removed SW1: SWITCH_HH, MOD_Footprints_Lib:SWITCH_HH_SK-13D26-G-6_5-K-GY, symbol SWITCH_1-3
- added P1: CONN_01X02, symbol CONN_01X02
- added P2: CONN_01X03, symbol CONN_01X03
- added SW1: SP3T, symbol SP3T
- C15, C9: value 100nF_X7R -> 100nF X7R
Connections:
- net labels added: +3.3VP, GNDD
- net labels removed: +3.3V, DGND
- wire segments 28 -> 29
Other:
- note added: "CHANNEL SELECTOR"
- note removed: "SWITCH H-H"
- moved on the sheet: C15, C9, R17, R18, R19, R23, R24, R25, R28
