File: hw-design/power.sch (KiCad schematic (older format))
At the start: 17 parts, among them CN1 CONN_PANNEL_2X2, CN2 CONN_PANNEL_2X2, U2 AP1117E50G, U3 AP1117E33G

Commit message: changing power schematic to use default kicad components library
Parts:
- removed CN1, CN2: CONN_PANNEL_2X2, MOD_Footprints_Lib:CONN_PANNEL, symbol CONN_PANNEL_2X2
- removed R11, R16: 0R, MOD_Footprints_Lib:SM0805, symbol R
- removed TP1, TP2: CONN_1, MOD_Footprints_Lib:SIL-1, symbol CONN_1
- removed U2: AP1117E50G, MOD_Footprints_Lib:SOT223_3, symbol LINEAR_REGULATOR_SOT223_3
- removed U3: AP1117E33G, MOD_Footprints_Lib:SOT223_3, symbol LINEAR_REGULATOR_SOT223_3
- added CN1, CN2: CONN_02X02, symbol CONN_02X02
- added TP1, TP2: ~, symbol CONN_01X01
- added U?: AP1117E50, symbol AP1117E50
- added U?: AP1117E33, symbol AP1117E33
- C2, C4, C8: value 100nF_X7R -> 100nF X7R
Connections:
- net labels added: +3.3VP, GNDD, VDD
- net labels removed: +3.3V, DGND, VCC
- wire segments 50 -> 42
Other:
- moved on the sheet: C1, C2, C3, C4, C7, C8, D1, RT1, RT2
