File: hw-design/board/control-chain.sch (KiCad schematic (older format))
At the start: 17 parts, among them J1 CC_INPUT, J2 CC_OUTPUT, Q4 2N7002, Q5 2N7002, Q6 IRFML8244TRPBF, U3 ISL83491

Commit message: fixing some footprints assignment
Parts:
- J1, J2: footprint MOD_Footprints:RJ45-RJHSE5084 -> Connect:RJHSE538X
Changed lines of the file:
@@
 F 0 "J1" H 3150 1500 50  0000 C CNN
 F 1 "CC_INPUT" H 3150 2400 50  0000 C CNN
-F 2 "MOD_Footprints:RJ45-RJHSE5084" H 3150 1950 60  0001 C CNN
+F 2 "Connect:RJHSE538X" H 3150 1950 60  0001 C CNN
 F 3 "" H 3150 1950 60  0000 C CNN
 F 4 "RJHSE-5381" H 0   0   50  0001 C CNN "MPN"
@@
 F 0 "J2" H 3150 3300 50  0000 C CNN
 F 1 "CC_OUTPUT" H 3150 4200 50  0000 C CNN
-F 2 "MOD_Footprints:RJ45-RJHSE5084" H 3150 3750 60  0001 C CNN
+F 2 "Connect:RJHSE538X" H 3150 3750 60  0001 C CNN
 F 3 "" H 3150 3750 60  0000 C CNN
 F 4 "RJHSE-5381" H 0   0   50  0001 C CNN "MPN"
